File: hardware/operacake/operacake.kicad_pcb (KiCad board)
At the start: 4 copper layers, 120 x 75 mm, 129 parts, among them J1 CONN_02X20, J2 CONN_02X20, P1 ADDRESS, P20 GPIO, P22 I2S, P28 SD, P9 BASEBAND, U1 MASWSS0129, U10 74LVC1G58, U11 74LVC1G58, U12 74LVC1G58, U13 74LVC1G58, U14 74AHC1G02, U15 74AHC1G02, U16 74LVC1G19, U2 SKY13322, U3 SKY13322, U4 PCA9557, U5 TC7MBL3245CFT, U6 74LVC1G58, U7 74LVC1G58, U8 74AHC1G08, U9 74AHC1G08

Commit message: brought master up to date
Parts:
- added C13: 33pF, gsg-modules:0402, F.Cu at (85.3, 132.6)
- added C14: 33pF, gsg-modules:0402, F.Cu at (80.1, 131.7)
- added C15: 33pF, gsg-modules:0402, F.Cu at (80.1, 129.5)
- added C16: 33pF, gsg-modules:0402, F.Cu at (85.6, 129.0)
- added C17: 33pF, gsg-modules:0402, F.Cu at (116.4, 167.7)
- added C18: 33pF, gsg-modules:0402, F.Cu at (123.6, 167.7)
- added C19: 33pF, gsg-modules:0402, F.Cu at (154.1, 129.3)
- added C20: 33pF, gsg-modules:0402, F.Cu at (159.6, 129.5)
- added C21: 33pF, gsg-modules:0402, F.Cu at (159.6, 131.7)
- added C22: 33pF, gsg-modules:0402, F.Cu at (154.2, 131.8)
- added C23: 100nF, gsg-modules:0402, F.Cu at (113.9, 129.3)
- added C24: 100nF, gsg-modules:0402, F.Cu at (124.4, 110.7)
- added C25: 100nF, gsg-modules:0402, F.Cu at (127.4, 116.9)
- added C26: 100nF, gsg-modules:0402, F.Cu at (127.3, 123.2)
- added C27: 100nF, gsg-modules:0402, F.Cu at (128.2, 130.3)
- added C28: 100nF, gsg-modules:0402, F.Cu at (114.0, 123.7)
- added C29: 100nF, gsg-modules:0402, F.Cu at (137.8, 108.3)
- added C30: 100nF, gsg-modules:0402, F.Cu at (131.8, 117.3)
- added C31: 100nF, gsg-modules:0402, F.Cu at (132.5, 123.1)
- added C32: 100nF, gsg-modules:0402, F.Cu at (132.0, 130.0)
- added C33: 100nF, gsg-modules:0402, F.Cu at (113.7, 134.7)
- added C34: 100nF, gsg-modules:0402, F.Cu at (132.0, 131.4)
- added C35: 100nF, gsg-modules:0402, F.Cu at (141.5, 126.5)
- C1, C10, C11, C12, C2, C3, C4, C5, C6, C7, C8, C9: value C -> 100nF
- moved U10 3.68 mm to (128.0, 113.3)
- moved U11 3.61 mm to (132.1, 113.4)
- moved U9 3.57 mm to (134.5, 109.5), turned to 270 degrees
- moved U8 2.45 mm to (127.8, 109.6), turned to 90 degrees
- moved U12 2.40 mm to (127.8, 119.6)
- moved U13 2.38 mm to (132.1, 119.6)
- moved TP23 2.32 mm to (162.0, 133.7)
- moved R12 2.10 mm to (130.8, 106.8)
- moved R14 2.10 mm to (134.8, 106.8)
- moved TP13 2.10 mm to (133.8, 104.3)
- moved TP2 2.04 mm to (163.1, 144.2)
- moved C10 1.64 mm to (123.9, 165.4)
- moved R11 1.55 mm to (140.6, 128.8)
- moved C9 1.44 mm to (115.1, 165.9)
- moved R10 1.26 mm to (130.7, 133.9), turned to 0 degrees
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Connections:
- J1 pad 10: (no net) -> Net-(J1-Pad10)
- J1 pad 11: (no net) -> Net-(J1-Pad11)
- J1 pad 12: (no net) -> Net-(J1-Pad12)
- J1 pad 13: (no net) -> Net-(J1-Pad13)
- J1 pad 14: (no net) -> Net-(J1-Pad14)
- J1 pad 15: (no net) -> Net-(J1-Pad15)
- J1 pad 16: (no net) -> Net-(J1-Pad16)
- J1 pad 17: (no net) -> Net-(J1-Pad17)
- J1 pad 18: (no net) -> Net-(J1-Pad18)
- J1 pad 19: (no net) -> Net-(J1-Pad19)
- J1 pad 20: (no net) -> Net-(J1-Pad20)
- J1 pad 21: (no net) -> Net-(J1-Pad21)
- J1 pad 22: (no net) -> Net-(J1-Pad22)
- J1 pad 23: (no net) -> Net-(J1-Pad23)
- J1 pad 24: (no net) -> Net-(J1-Pad24)
- J1 pad 25: (no net) -> Net-(J1-Pad25)
- J1 pad 26: (no net) -> Net-(J1-Pad26)
- J1 pad 27: (no net) -> Net-(J1-Pad27)
- J1 pad 28: (no net) -> Net-(J1-Pad28)
- J1 pad 29: (no net) -> Net-(J1-Pad29)
- J1 pad 3: (no net) -> Net-(J1-Pad3)
- J1 pad 30: (no net) -> Net-(J1-Pad30)
- J1 pad 31: (no net) -> Net-(J1-Pad31)
- J1 pad 32: (no net) -> Net-(J1-Pad32)
- J1 pad 33: (no net) -> Net-(J1-Pad33)
- J1 pad 34: (no net) -> Net-(J1-Pad34)
- J1 pad 35: (no net) -> Net-(J1-Pad35)
- J1 pad 36: (no net) -> Net-(J1-Pad36)
- J1 pad 37: (no net) -> Net-(J1-Pad37)
- J1 pad 38: (no net) -> Net-(J1-Pad38)
- J1 pad 39: (no net) -> Net-(J1-Pad39)
- J1 pad 4: (no net) -> Net-(J1-Pad4)
- J1 pad 40: (no net) -> Net-(J1-Pad40)
- J1 pad 5: (no net) -> Net-(J1-Pad5)
- J1 pad 6: (no net) -> Net-(J1-Pad6)
- J1 pad 7: (no net) -> Net-(J1-Pad7)
- J1 pad 8: (no net) -> Net-(J1-Pad8)
- J1 pad 9: (no net) -> Net-(J1-Pad9)
- J2 pad 11: (no net) -> Net-(J2-Pad11)
- J2 pad 12: (no net) -> Net-(J2-Pad12)
- J2 pad 13: (no net) -> Net-(J2-Pad13)
- J2 pad 14: (no net) -> Net-(J2-Pad14)
- J2 pad 15: (no net) -> Net-(J2-Pad15)
- J2 pad 16: (no net) -> Net-(J2-Pad16)
- J2 pad 17: (no net) -> Net-(J2-Pad17)
- J2 pad 18: (no net) -> Net-(J2-Pad18)
- J2 pad 19: (no net) -> Net-(J2-Pad19)
- J2 pad 2: (no net) -> Net-(J2-Pad2)
- J2 pad 20: (no net) -> Net-(J2-Pad20)
- J2 pad 21: (no net) -> Net-(J2-Pad21)
- J2 pad 22: (no net) -> Net-(J2-Pad22)
- J2 pad 23: (no net) -> Net-(J2-Pad23)
- J2 pad 24: (no net) -> Net-(J2-Pad24)
- J2 pad 25: (no net) -> Net-(J2-Pad25)
- J2 pad 26: (no net) -> Net-(J2-Pad26)
- J2 pad 27: (no net) -> Net-(J2-Pad27)
- J2 pad 28: (no net) -> Net-(J2-Pad28)
- J2 pad 29: (no net) -> Net-(J2-Pad29)
- J2 pad 3: (no net) -> Net-(J2-Pad3)
- J2 pad 30: (no net) -> Net-(J2-Pad30)
- J2 pad 31: (no net) -> Net-(J2-Pad31)
- J2 pad 32: (no net) -> Net-(J2-Pad32)
- J2 pad 33: (no net) -> Net-(J2-Pad33)
- J2 pad 34: (no net) -> Net-(J2-Pad34)
- J2 pad 35: (no net) -> Net-(J2-Pad35)
- J2 pad 36: (no net) -> Net-(J2-Pad36)
- J2 pad 37: (no net) -> Net-(J2-Pad37)
- J2 pad 38: (no net) -> Net-(J2-Pad38)
- J2 pad 4: (no net) -> Net-(J2-Pad4)
- J2 pad 5: (no net) -> Net-(J2-Pad5)
- P20 pad 1: (no net) -> Net-(P20-Pad1)
- P20 pad 13: GND -> Net-(P20-Pad13)
- P20 pad 14: (no net) -> Net-(P20-Pad14)
- P20 pad 16: (no net) -> Net-(P20-Pad16)
- P20 pad 17: (no net) -> Net-(P20-Pad17)
- P20 pad 18: (no net) -> Net-(P20-Pad18)
- P20 pad 2: (no net) -> Net-(P20-Pad2)
- P20 pad 20: (no net) -> Net-(P20-Pad20)
- P20 pad 21: (no net) -> Net-(P20-Pad21)
- P20 pad 22: (no net) -> Net-(P20-Pad22)
- P20 pad 4: (no net) -> Net-(P20-Pad4)
- P20 pad 6: (no net) -> Net-(P20-Pad6)
- P20 pad 7: (no net) -> Net-(P20-Pad7)
- P20 pad 8: (no net) -> Net-(P20-Pad8)
- P22 pad 1: (no net) -> Net-(P22-Pad1)
- P22 pad 12: (no net) -> Net-(P22-Pad12)
- P22 pad 13: (no net) -> Net-(P22-Pad13)
- P22 pad 14: (no net) -> Net-(P22-Pad14)
- P22 pad 15: (no net) -> Net-(P22-Pad15)
- P22 pad 16: (no net) -> Net-(P22-Pad16)
- P22 pad 17: (no net) -> Net-(P22-Pad17)
- P22 pad 19: (no net) -> Net-(P22-Pad19)
- P22 pad 2: (no net) -> Net-(P22-Pad2)
- P22 pad 20: (no net) -> Net-(P22-Pad20)
- P22 pad 21: (no net) -> Net-(P22-Pad21)
- P22 pad 22: (no net) -> Net-(P22-Pad22)
- P22 pad 23: (no net) -> Net-(P22-Pad23)
- P22 pad 25: (no net) -> Net-(P22-Pad25)
- P22 pad 3: (no net) -> Net-(P22-Pad3)
- P22 pad 5: (no net) -> Net-(P22-Pad5)
- P22 pad 6: (no net) -> Net-(P22-Pad6)
- P22 pad 7: (no net) -> Net-(P22-Pad7)
- P22 pad 8: (no net) -> Net-(P22-Pad8)
- P22 pad 9: (no net) -> Net-(P22-Pad9)
- P28 pad 10: (no net) -> Net-(P28-Pad10)
- P28 pad 11: (no net) -> Net-(P28-Pad11)
- P28 pad 13: (no net) -> Net-(P28-Pad13)
- P28 pad 14: (no net) -> Net-(P28-Pad14)
- P28 pad 15: (no net) -> Net-(P28-Pad15)
- P28 pad 16: (no net) -> Net-(P28-Pad16)
- P28 pad 17: (no net) -> Net-(P28-Pad17)
- P28 pad 18: (no net) -> Net-(P28-Pad18)
- P28 pad 19: (no net) -> Net-(P28-Pad19)
- P28 pad 20: (no net) -> Net-(P28-Pad20)
- P28 pad 21: (no net) -> Net-(P28-Pad21)
- P28 pad 22: (no net) -> Net-(P28-Pad22)
- P28 pad 3: (no net) -> Net-(P28-Pad3)
- P28 pad 4: (no net) -> Net-(P28-Pad4)
- P28 pad 5: (no net) -> Net-(P28-Pad5)
- P28 pad 6: (no net) -> Net-(P28-Pad6)
- P28 pad 7: (no net) -> Net-(P28-Pad7)
- P28 pad 8: (no net) -> Net-(P28-Pad8)
- P28 pad 9: (no net) -> Net-(P28-Pad9)
- P9 pad 10: (no net) -> Net-(P9-Pad10)
- P9 pad 11: (no net) -> Net-(P9-Pad11)
- P9 pad 12: (no net) -> Net-(P9-Pad12)
- P9 pad 13: (no net) -> Net-(P9-Pad13)
- P9 pad 4: (no net) -> Net-(P9-Pad4)
- P9 pad 5: (no net) -> Net-(P9-Pad5)
- P9 pad 6: (no net) -> Net-(P9-Pad6)
- P9 pad 7: (no net) -> Net-(P9-Pad7)
- U2 pad 3: (no net) -> Net-(U2-Pad3)
- U3 pad 3: (no net) -> Net-(U3-Pad3)
- U5 pad 1: (no net) -> Net-(U5-Pad1)
- U5 pad 11: (no net) -> Net-(U5-Pad11)
- U5 pad 12: (no net) -> Net-(U5-Pad12)
- U5 pad 13: (no net) -> Net-(U5-Pad13)
- U5 pad 7: (no net) -> Net-(U5-Pad7)
- U5 pad 8: (no net) -> Net-(U5-Pad8)
- U5 pad 9: (no net) -> Net-(U5-Pad9)
Routing:
- net GND: track 55.6 -> 92.6 mm, vias 29 -> 52
- net VCC: track 34.9 -> 52.0 mm
- net /U3V3: track 75.8 -> 65.4 mm
- net /U3CTRL1: track 38.1 -> 45.4 mm, vias 1 -> 3
- net /U2CTRL0: track 62.2 -> 69.0 mm, vias 1 -> 3
- net /U1VC1: track 54.0 -> 60.1 mm, vias 2 -> 4
- net /U2V2: track 82.1 -> 86.6 mm, vias 3 -> 5
- net Net-(R2-Pad2): track 6.15 -> 10.1 mm
- net /U2V1: track 86.6 -> 90.0 mm
- net /U3V2: track 73.5 -> 76.8 mm
- net /U2V4: track 84.1 -> 87.3 mm, vias 4 -> 2
- net /U2CTRL1: track 39.0 -> 41.9 mm
- net /!RESET: track 6.78 -> 9.48 mm
- net Net-(DA0-Pad1): track 86.5 -> 89.1 mm
- net Net-(C9-Pad1): track 3.09 -> 5.14 mm
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Other:
- board text added: "30 October 2018"
- board text added: "A3"
- board text added: "A4"
- board text added: "B0"
- board text added: "B1"
- board text added: "B2"
- board text added: "B3"
- board text added: "B4"
- board text added: "https://greatscottgadgets.com/hackrf/"
- board text removed: "4 October 2016"
- board text removed: "PA0"
- board text removed: "PA1"
- board text removed: "PA2"
- board text removed: "PA3"
- board text removed: "PA4"
- board text removed: "PB0"
- board text removed: "PB1"
- board text removed: "PB2"
- board text removed: "PB3"
- board text removed: "PB4"
- board text removed: "http://greatscottgadgets.com/hackrf/"
